File: FusionX/LCD.kicad_sch (KiCad schematic)
At the start: 1 part, among them J1 MainLCD

Commit message: Updated sheet
Other:
- company: (none) -> NoahGWood
- title: (none) -> FusionX
Changed lines of the file:
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@@
 (kicad_sch (version 20230121) (generator eeschema)
   (paper "A4")
+  (title_block
+    (title "FusionX")
+    (date "2023-08-15")
+    (rev "1")
+    (company "NoahGWood")
+    (comment 1 "License: The Unlicense")
+    (comment 2 "twitch.tv/u/noahgwood")
+    (comment 3 "Developed Live On:")
+    (comment 4 "SC600Y Based Smartphone")
+  )
   (junction (at 66.04 66.04) (diameter 0) (color 0 0 0 0)
   )
