File: FusionX/power.kicad_sch (KiCad schematic)
At the start: 8 parts, among them J2 BAT, P1 USB_C_Plug

Commit message: Updated sheet
Other:
- company: (none) -> NoahGWood
Changed lines of the file:
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@@
     (date "2023-08-15")
     (rev "1")
+    (company "NoahGWood")
     (comment 1 "License: The Unlicense")
+    (comment 2 "twitch.tv/u/noahgwood")
+    (comment 3 "Developed Live On:")
     (comment 4 "SC600Y Based Smartphone")
   )

Commit message: Finished RaspiLCD Added Antennas Started secondary LCD
Changed lines of the file:
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@@
     (stroke (width 0) (type default))
   )
-  (text_box "TODO:\n	Find MUX/DEMUX for USB 3.0\n	"
+  (text_box "TODO:\n	Find MUX/DEMUX for USB 3.0\n	3.3v Regulator"
     (at 107.95 95.25 0) (size 109.855 53.34)
     (stroke (width 0) (type default))

Commit message: Implemented: 	USB-C Super Speed 	Capacitve Touch Screen 	Secondary LCD
Started On:
	PCB Layout
	Case Design
Parts:
- removed P1: USB_C_Plug, symbol Connector:USB_C_Plug
- J2: footprint (none) -> Connector_JST:JST_PH_B2B-PH-K_1x02_P2.00mm_Vertical
Changed lines of the file:
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@@
   (title_block
     (title "FusionX")
-    (date "2023-08-15")
+    (date "2023-08-17")
     (rev "1")
     (company "NoahGWood")
@@
   (junction (at 52.07 40.64) (diameter 0) (color 0 0 0 0)
   )
-  (junction (at 56.515 156.845) (diameter 0) (color 0 0 0 0)
-  )
   (junction (at 83.82 40.64) (diameter 0) (color 0 0 0 0)
   )
@@
     (stroke (width 0) (type default))
   )
-  (wire (pts (xy 56.515 156.845) (xy 60.325 156.845))
-    (stroke (width 0) (type default))
-  )
   (wire (pts (xy 52.07 55.88) (xy 46.99 55.88))
     (stroke (width 0) (type default))
   )
-  (wire (pts (xy 52.705 156.845) (xy 56.515 156.845))
-    (stroke (width 0) (type default))
-  )
   (wire (pts (xy 52.07 55.88) (xy 52.07 57.15))
     (stroke (width 0) (type default))
@@
     (stroke (width 0) (type default))
   )
-  (text_box "TODO:\n	Find MUX/DEMUX for USB 3.0\n	3.3v Regulator"
+  (text_box "TODO:\n	3.3v Regulator"
     (at 107.95 95.25 0) (size 109.855 53.34)
     (stroke (width 0) (type default))
@@
     )
   )
-  (symbol (lib_id "power:GND") (at 56.515 156.845 0) (unit 1)
-    (in_bom yes) (on_board yes) (dnp no) (fields_autoplaced)
-    (property "Reference" "#PWR05" (at 56.515 163.195 0)
-      (effects (font (size 1.27 1.27)) hide)
-    )
-    (property "Value" "GND" (at 56.515 161.29 0)
-      (effects (font (size 1.27 1.27)))
-    )
-    (property "Footprint" "" (at 56.515 156.845 0)
-      (effects (font (size 1.27 1.27)) hide)
-    )
-    (property "Datasheet" "" (at 56.515 156.845 0)
-      (effects (font (size 1.27 1.27)) hide)
-    )
-    (pin "1")
-    (instances
-      (project "FusionX"
-        (path "/91d1c248-6dd5-47d7-a0ee-1ed6541bbbfb/1984d1b6-a445-4aa7-9bc2-a44faa93b5d0"
-          (reference "#PWR05") (unit 1)
-        )
-      )
-    )
-  )
   (symbol (lib_id "Device:C_Small") (at 71.12 43.18 0) (unit 1)
     (in_bom yes) (on_board yes) (dnp no) (fields_autoplaced)
@@
       (effects (font (size 1.27 1.27)))
     )
-    (property "Footprint" "" (at 34.29 41.91 0)
+    (property "Footprint" "Connector_JST:JST_PH_B2B-PH-K_1x02_P2.00mm_Vertical" (at 34.29 41.91 0)
       (effects (font (size 1.27 1.27)) hide)
     )
@@
         )
       )
-    )
-  )
-  (symbol (lib_id "Connector:USB_C_Plug") (at 60.325 116.205 0) (unit 1)
-    (in_bom yes) (on_board yes) (dnp no) (fields_autoplaced)
-    (property "Reference" "P1" (at 60.325 83.82 0)
-      (effects (font (size 1.27 1.27)))
-    )
-    (property "Value" "USB_C_Plug" (at 60.325 86.36 0)
-      (effects (font (size 1.27 1.27)))
-    )
-    (property "Footprint" "" (at 64.135 116.205 0)
-      (effects (font (size 1.27 1.27)) hide)
-    )
-    (property "Datasheet" "https://www.usb.org/sites/default/files/documents/usb_type-c.zip" (at 64.135 116.205 0)
-      (effects (font (size 1.27 1.27)) hide)
-    )
-    (pin "A1")
-    (pin "A10")
-    (pin "A11")
-    (pin "A12")
-    (pin "A2")
-    (pin "A3")
-    (pin "A4")
-    (pin "A5")
-    (pin "A6")
-    (pin "A7")
-    (pin "A8")
-    (pin "A9")
-    (pin "B1")
-    (pin "B10")
-    (pin "B11")
-    (pin "B12")
-    (pin "B2")
-    (pin "B3")
-    (pin "B4")
-    (pin "B5")
-    (pin "B8")
-    (pin "B9")
-    (pin "S1")
-    (instances
-      (project "FusionX"
-        (path "/91d1c248-6dd5-47d7-a0ee-1ed6541bbbfb/1984d1b6-a445-4aa7-9bc2-a44faa93b5d0"
-          (reference "P1") (unit 1)
-        )
-      )
